File: hdmi_TXn.sch (KiCad schematic (older format))
At the start: 21 parts

Commit message: Make sure the schematic has leading zeros.
Parts:
- renumbered C$TXn$1 to C$TXn$01, C$TXn$2 to C$TXn$02, C$TXn$3 to C$TXn$03, C$TXn$4 to C$TXn$04, C$TXn$5 to C$TXn$05, C$TXn$6 to C$TXn$06, C$TXn$7 to C$TXn$07, C$TXn$8 to C$TXn$08, D$TXn$1 to D$TXn$01, P$TXn$1 to P$TXn$01, R$TXn$1 to R$TXn$01, R$TXn$2 to R$TXn$02, R$TXn$3 to R$TXn$03, R$TXn$4 to R$TXn$04, R$TXn$5 to R$TXn$05, R$TXn$8 to R$TXn$08
Changed lines of the file:
@@
 $EndComp
 $Comp
-L DIODE D$TXn$1
+L DIODE D$TXn$01
 U 1 1 57C0774F
 P 10600 5450
-F 0 "D$TXn$1" H 10600 5550 50  0000 C CNN
+F 0 "D$TXn$01" H 10600 5550 50  0000 C CNN
 F 1 "DIODE" H 10600 5350 50  0000 C CNN
 F 2 "" H 10600 5450 60  0001 C CNN
@@
 $EndComp
 $Comp
-L R R$TXn$8
+L R R$TXn$08
 U 1 1 57C07751
 P 10600 4950
-AR Path="/57C07751" Ref="R$TXn$8"  Part="1"
-AR Path="/57C01383/57C07751" Ref="R$TXn$3"  Part="1"
-F 0 "R$TXn$8" V 10700 4950 50  0000 C CNN
+AR Path="/57C07751" Ref="R$TXn$08"  Part="1"
+AR Path="/57C01383/57C07751" Ref="R$TXn$03"  Part="1"
+F 0 "R$TXn$08" V 10700 4950 50  0000 C CNN
 F 1 "R" V 10607 4951 50  0000 C CNN
 F 2 "Resistors_SMD:R_0402" V 10530 4950 30  0001 C CNN
@@
 $EndComp
 $Comp
-L R R$TXn$2
+L R R$TXn$02
 U 1 1 57C07753
 P 3900 4400
-AR Path="/57C07753" Ref="R$TXn$2"  Part="1"
-AR Path="/57C01383/57C07753" Ref="R$TXn$1"  Part="1"
-F 0 "R$TXn$2" V 3800 4400 50  0000 C CNN
+AR Path="/57C07753" Ref="R$TXn$02"  Part="1"
+AR Path="/57C01383/57C07753" Ref="R$TXn$01"  Part="1"
+F 0 "R$TXn$02" V 3800 4400 50  0000 C CNN
 F 1 "2k2" V 3907 4401 50  0000 C CNN
 F 2 "Resistors_SMD:R_0402" V 3830 4400 30  0001 C CNN
@@
 $EndComp
 $Comp
-L R R$TXn$1
+L R R$TXn$01
 U 1 1 57C07755
 P 4000 4400
-AR Path="/57C07755" Ref="R$TXn$1"  Part="1"
-AR Path="/57C01383/57C07755" Ref="R$TXn$2"  Part="1"
-F 0 "R$TXn$1" V 4080 4400 50  0000 C CNN
+AR Path="/57C07755" Ref="R$TXn$01"  Part="1"
+AR Path="/57C01383/57C07755" Ref="R$TXn$02"  Part="1"
+F 0 "R$TXn$01" V 4080 4400 50  0000 C CNN
 F 1 "2k2" V 4007 4401 50  0000 C CNN
 F 2 "Resistors_SMD:R_0402" V 3930 4400 30  0001 C CNN
@@
 	5700 6600 6750 6600
 $Comp
-L Csmall C$TXn$1
+L Csmall C$TXn$01
 U 1 1 57B7CD9B
 P 6300 4800
-F 0 "C$TXn$1" V 6265 4840 30  0000 L CNN
+F 0 "C$TXn$01" V 6265 4840 30  0000 L CNN
 F 1 "100n" V 6270 4665 30  0000 L CNN
 F 2 "Capacitors_SMD:C_0402" H 6300 4800 60  0001 C CNN
@@
 $EndComp
 $Comp
-L Csmall C$TXn$2
+L Csmall C$TXn$02
 U 1 1 57C07759
 P 6300 4900
-F 0 "C$TXn$2" V 6270 4940 30  0000 L CNN
+F 0 "C$TXn$02" V 6270 4940 30  0000 L CNN
 F 1 "100n" V 6270 4765 30  0000 L CNN
 F 2 "Capacitors_SMD:C_0402" H 6300 4900 60  0001 C CNN
@@
 HDMIP_$TXn$_SDA
 $Comp
-L R R$TXn$4
+L R R$TXn$04
 U 1 1 57C07769
 P 3900 5600
-AR Path="/57C07769" Ref="R$TXn$4"  Part="1"
-AR Path="/57C01383/57C07769" Ref="R$TXn$4"  Part="1"
-F 0 "R$TXn$4" V 3800 5600 50  0000 C CNN
+AR Path="/57C07769" Ref="R$TXn$04"  Part="1"
+AR Path="/57C01383/57C07769" Ref="R$TXn$04"  Part="1"
+F 0 "R$TXn$04" V 3800 5600 50  0000 C CNN
 F 1 "2k2" V 3907 5601 50  0000 C CNN
 F 2 "Resistors_SMD:R_0402" V 3830 5600 30  0001 C CNN
@@
 $EndComp
 $Comp
-L R R$TXn$5
+L R R$TXn$05
 U 1 1 57B7FCE7
 P 4000 5600
-AR Path="/57B7FCE7" Ref="R$TXn$5"  Part="1"
-AR Path="/57C01383/57B7FCE7" Ref="R$TXn$5"  Part="1"
-F 0 "R$TXn$5" V 4080 5600 50  0000 C CNN
+AR Path="/57B7FCE7" Ref="R$TXn$05"  Part="1"
+AR Path="/57C01383/57B7FCE7" Ref="R$TXn$05"  Part="1"
+F 0 "R$TXn$05" V 4080 5600 50  0000 C CNN
 F 1 "2k2" V 4007 5601 50  0000 C CNN
 F 2 "Resistors_SMD:R_0402" V 3930 5600 30  0001 C CNN
@@
 HDMI_$TXn$_SDA
 $Comp
-L R R$TXn$3
+L R R$TXn$03
 U 1 1 57C0776D
 P 6500 6900
-AR Path="/57C0776D" Ref="R$TXn$3"  Part="1"
-AR Path="/57C01383/57C0776D" Ref="R$TXn$6"  Part="1"
-F 0 "R$TXn$3" V 6580 6900 50  0000 C CNN
+AR Path="/57C0776D" Ref="R$TXn$03"  Part="1"
+AR Path="/57C01383/57C0776D" Ref="R$TXn$06"  Part="1"
+F 0 "R$TXn$03" V 6580 6900 50  0000 C CNN
 F 1 "12k4" V 6507 6901 50  0000 C CNN
 F 2 "Resistors_SMD:R_0402" V 6430 6900 30  0001 C CNN
@@
 P 8500 3850
 AR Path="/57C07777" Ref="C$TXn$17"  Part="1"
-AR Path="/57C01383/57C07777" Ref="C$TXn$2"  Part="1"
+AR Path="/57C01383/57C07777" Ref="C$TXn$02"  Part="1"
 F 0 "C$TXn$17" H 8300 3750 30  0000 L CNN
 F 1 "100n" H 8300 3850 30  0000 L CNN
@@
 P 8300 3850
 AR Path="/57C07779" Ref="C$TXn$16"  Part="1"
-AR Path="/57C01383/57C07779" Ref="C$TXn$1"  Part="1"
+AR Path="/57C01383/57C07779" Ref="C$TXn$01"  Part="1"
 F 0 "C$TXn$16" H 8350 3750 30  0000 L CNN
 F 1 "100n" H 8400 3850 30  0000 L CNN
@@
 HDMI_$TXn$_CEC
 $Comp
-L CONN_02X06 P$TXn$1
+L CONN_02X06 P$TXn$01
 U 1 1 57D65C54
 P 3415 6820
-F 0 "P$TXn$1" H 3415 7285 50  0000 C CNN
+F 0 "P$TXn$01" H 3415 7285 50  0000 C CNN
 F 1 "CONN_02X06" H 3415 7194 50  0000 C CNN
 F 2 "Pin_Headers:Pin_Header_Straight_2x06" H 3415 5620 50  0001 C CNN
@@
 HDMI_$TXn$_EQ0
 $Comp
-L Csmall C$TXn$3
+L Csmall C$TXn$03
 U 1 1 57D7B3E7
 P 6300 5100
-F 0 "C$TXn$3" V 6265 5140 30  0000 L CNN
+F 0 "C$TXn$03" V 6265 5140 30  0000 L CNN
 F 1 "100n" V 6270 4965 30  0000 L CNN
 F 2 "Capacitors_SMD:C_0402" H 6300 5100 60  0001 C CNN
@@
 $EndComp
 $Comp
-L Csmall C$TXn$4
+L Csmall C$TXn$04
 U 1 1 57D7B3EF
 P 6300 5200
-F 0 "C$TXn$4" V 6270 5240 30  0000 L CNN
+F 0 "C$TXn$04" V 6270 5240 30  0000 L CNN
 F 1 "100n" V 6270 5065 30  0000 L CNN
 F 2 "Capacitors_SMD:C_0402" H 6300 5200 60  0001 C CNN
@@
 $EndComp
 $Comp
-L Csmall C$TXn$5
+L Csmall C$TXn$05
 U 1 1 57D7B73E
 P 6300 5400
-F 0 "C$TXn$5" V 6265 5440 30  0000 L CNN
+F 0 "C$TXn$05" V 6265 5440 30  0000 L CNN
 F 1 "100n" V 6270 5265 30  0000 L CNN
 F 2 "Capacitors_SMD:C_0402" H 6300 5400 60  0001 C CNN
@@
 $EndComp
 $Comp
-L Csmall C$TXn$6
+L Csmall C$TXn$06
 U 1 1 57D7B746
 P 6300 5500
-F 0 "C$TXn$6" V 6270 5540 30  0000 L CNN
+F 0 "C$TXn$06" V 6270 5540 30  0000 L CNN
 F 1 "100n" V 6270 5365 30  0000 L CNN
 F 2 "Capacitors_SMD:C_0402" H 6300 5500 60  0001 C CNN
@@
 $EndComp
 $Comp
-L Csmall C$TXn$7
+L Csmall C$TXn$07
 U 1 1 57D7B74E
 P 6300 5700
-F 0 "C$TXn$7" V 6265 5740 30  0000 L CNN
+F 0 "C$TXn$07" V 6265 5740 30  0000 L CNN
 F 1 "100n" V 6270 5565 30  0000 L CNN
 F 2 "Capacitors_SMD:C_0402" H 6300 5700 60  0001 C CNN
@@
 $EndComp
 $Comp
-L Csmall C$TXn$8
+L Csmall C$TXn$08
 U 1 1 57D7B756
 P 6300 5800
-F 0 "C$TXn$8" V 6270 5840 30  0000 L CNN
+F 0 "C$TXn$08" V 6270 5840 30  0000 L CNN
 F 1 "100n" V 6270 5665 30  0000 L CNN
 F 2 "Capacitors_SMD:C_0402" H 6300 5800 60  0001 C CNN

Commit message: Always have a prefix 1.
Parts:
- renumbered C$TXn$01 to C$TXn$101, C$TXn$02 to C$TXn$102, C$TXn$03 to C$TXn$103, C$TXn$04 to C$TXn$104, C$TXn$05 to C$TXn$105, C$TXn$06 to C$TXn$106, C$TXn$07 to C$TXn$107, C$TXn$08 to C$TXn$108, C$TXn$13 to C$TXn$113, C$TXn$16 to C$TXn$116, C$TXn$17 to C$TXn$117, D$TXn$01 to D$TXn$101, J$TXn$1 to J$TXn$11, P$TXn$01 to P$TXn$101, R$TXn$01 to R$TXn$101, R$TXn$02 to R$TXn$102, R$TXn$03 to R$TXn$103, R$TXn$04 to R$TXn$104, R$TXn$05 to R$TXn$105, R$TXn$08 to R$TXn$108, U$TXn$1 to U$TXn$11
Connections:
- net labels added: $TXn$15V0, HDMIP_$TXn$1_D1+, HDMIP_$TXn$1_D1-, HDMIP_$TXn$1_D2+, HDMIP_$TXn$1_D2-, HDMIP_$TXn$1_D3+, HDMIP_$TXn$1_D3-, HDMIP_$TXn$1_D4+, HDMIP_$TXn$1_D4-, HDMIP_$TXn$1_HPD, HDMIP_$TXn$1_SCL, HDMIP_$TXn$1_SDA, HDMI_$TXn$1_CEC, HDMI_$TXn$1_D1+, HDMI_$TXn$1_D1-, HDMI_$TXn$1_D2+, HDMI_$TXn$1_D2-, HDMI_$TXn$1_D3+, HDMI_$TXn$1_D3-, HDMI_$TXn$1_D4+, HDMI_$TXn$1_D4-, HDMI_$TXn$1_DDC_EN, HDMI_$TXn$1_DDET, HDMI_$TXn$1_EQ0, HDMI_$TXn$1_EQ1, HDMI_$TXn$1_HIZ_EN, HDMI_$TXn$1_HPD, HDMI_$TXn$1_SCL, HDMI_$TXn$1_SDA, ~HDMI_$TXn$1_OE
- net labels removed: $TXn$5V0, HDMIP_$TXn$_D1+, HDMIP_$TXn$_D1-, HDMIP_$TXn$_D2+, HDMIP_$TXn$_D2-, HDMIP_$TXn$_D3+, HDMIP_$TXn$_D3-, HDMIP_$TXn$_D4+, HDMIP_$TXn$_D4-, HDMIP_$TXn$_HPD, HDMIP_$TXn$_SCL, HDMIP_$TXn$_SDA, HDMI_$TXn$_CEC, HDMI_$TXn$_D1+, HDMI_$TXn$_D1-, HDMI_$TXn$_D2+, HDMI_$TXn$_D2-, HDMI_$TXn$_D3+, HDMI_$TXn$_D3-, HDMI_$TXn$_D4+, HDMI_$TXn$_D4-, HDMI_$TXn$_DDC_EN, HDMI_$TXn$_DDET, HDMI_$TXn$_EQ0, HDMI_$TXn$_EQ1, HDMI_$TXn$_HIZ_EN, HDMI_$TXn$_HPD, HDMI_$TXn$_SCL, HDMI_$TXn$_SDA, ~HDMI_$TXn$_OE
