File: hdmi_TXn.sch (KiCad schematic (older format))
At the start: 21 parts

Commit message: Small fixes to major component numbers.
Parts:
- renumbered J$TXn$11 to J$TXn$1, P$TXn$101 to P$TXn$1, U$TXn$11 to U$TXn$1
Changed lines of the file:
@@
 $EndDescr
 $Comp
-L PTN3363 U$TXn$11
+L PTN3363 U$TXn$1
 U 1 1 57C07746
 P 7450 5400
-F 0 "U$TXn$11" H 7100 6900 60  0000 C CNN
+F 0 "U$TXn$1" H 7100 6900 60  0000 C CNN
 F 1 "PTN3363" H 7700 3950 60  0000 C CNN
 F 2 "Housings_DFN_QFN:QFN-32-1EP_5x5mm_Pitch0.5mm" H 7350 5600 60  0001 C CNN
@@
 $EndComp
 $Comp
-L HDMI J$TXn$11
+L HDMI J$TXn$1
 U 1 1 57B7B39B
 P 12300 5650
-F 0 "J$TXn$11" H 12100 6700 60  0000 C CNN
+F 0 "J$TXn$1" H 12100 6700 60  0000 C CNN
 F 1 "HDMI" V 12450 5650 60  0000 C CNN
 F 2 "" H 12250 5650 60  0001 C CNN
@@
 HDMI_$TXn$1_CEC
 $Comp
-L CONN_02X06 P$TXn$101
+L CONN_02X06 P$TXn$1
 U 1 1 57D65C54
 P 3415 6820
-F 0 "P$TXn$101" H 3415 7285 50  0000 C CNN
+F 0 "P$TXn$1" H 3415 7285 50  0000 C CNN
 F 1 "CONN_02X06" H 3415 7194 50  0000 C CNN
 F 2 "Pin_Headers:Pin_Header_Straight_2x06" H 3415 5620 50  0001 C CNN

Commit message: Fix caps in HDMI Tx template
Parts:
- C$TXn$101, C$TXn$102, C$TXn$103, C$TXn$104, C$TXn$105, C$TXn$106, C$TXn$107, C$TXn$108: symbol Csmall -> C_Small
Changed lines of the file:
@@
 	5700 6600 6750 6600
 $Comp
-L Csmall C$TXn$101
+L C_Small C$TXn$101
 U 1 1 57B7CD9B
 P 6300 4800
@@
 $EndComp
 $Comp
-L Csmall C$TXn$102
+L C_Small C$TXn$102
 U 1 1 57C07759
 P 6300 4900
@@
 HDMI_$TXn$1_EQ0
 $Comp
-L Csmall C$TXn$103
+L C_Small C$TXn$103
 U 1 1 57D7B3E7
 P 6300 5100
@@
 $EndComp
 $Comp
-L Csmall C$TXn$104
+L C_Small C$TXn$104
 U 1 1 57D7B3EF
 P 6300 5200
@@
 $EndComp
 $Comp
-L Csmall C$TXn$105
+L C_Small C$TXn$105
 U 1 1 57D7B73E
 P 6300 5400
@@
 $EndComp
 $Comp
-L Csmall C$TXn$106
+L C_Small C$TXn$106
 U 1 1 57D7B746
 P 6300 5500
@@
 $EndComp
 $Comp
-L Csmall C$TXn$107
+L C_Small C$TXn$107
 U 1 1 57D7B74E
 P 6300 5700
@@
 $EndComp
 $Comp
-L Csmall C$TXn$108
+L C_Small C$TXn$108
 U 1 1 57D7B756
 P 6300 5800

Commit message: Add 5V regulator for HDMI Tx in template
Parts:
- added C$TXn$109: 0.33uF, symbol C
- added C$TXn$110, C$TXn$111: 0.1uF, symbol C
- added R$TXn$106: 100K, symbol R
- added U$TXn$101: ΜA78L00, symbol ΜA78L00
Connections:
- net labels added: VCC12V0
- wire segments 109 -> 123
Changed lines of the file:
@@
 HDMIP_$TXn$1_HPD
 $Comp
-L GND #PWR01
+L GND #PWR106
 U 1 1 57B7C214
 P 7450 7150
-F 0 "#PWR01" H 7450 6900 60  0001 C CNN
+F 0 "#PWR106" H 7450 6900 60  0001 C CNN
 F 1 "GND" H 7450 7000 60  0000 C CNN
 F 2 "" H 7450 7150 60  0000 C CNN
@@
 $EndComp
 $Comp
-L GND #PWR02
+L GND #PWR112
 U 1 1 57C0774B
 P 11600 6900
-F 0 "#PWR02" H 11600 6650 60  0001 C CNN
+F 0 "#PWR112" H 11600 6650 60  0001 C CNN
 F 1 "GND" H 11600 6750 60  0000 C CNN
 F 2 "" H 11600 6900 60  0000 C CNN
@@
 $EndComp
 $Comp
-L VCC3V3 #PWR03
+L VCC3V3 #PWR105
 U 1 1 57B7C310
 P 7450 3600
-F 0 "#PWR03" H 7450 3450 60  0001 C CNN
+F 0 "#PWR105" H 7450 3450 60  0001 C CNN
 F 1 "VCC3V3" H 7450 3740 60  0000 C CNN
 F 2 "" H 7450 3600 60  0000 C CNN
@@
 	4000 4100 4000 4250
 $Comp
-L VCC3V3 #PWR04
+L VCC3V3 #PWR103
 U 1 1 57C07768
 P 3950 4050
-F 0 "#PWR04" H 3950 3900 60  0001 C CNN
+F 0 "#PWR103" H 3950 3900 60  0001 C CNN
 F 1 "VCC3V3" H 3950 4190 60  0000 C CNN
 F 2 "" H 3950 4050 60  0000 C CNN
@@
 	6500 6300 6500 6750
 $Comp
-L GND #PWR05
+L GND #PWR104
 U 1 1 57C0776F
 P 6500 7150
-F 0 "#PWR05" H 6500 6900 60  0001 C CNN
+F 0 "#PWR104" H 6500 6900 60  0001 C CNN
 F 1 "GND" H 6500 7000 60  0000 C CNN
 F 2 "" H 6500 7150 60  0000 C CNN
@@
 HDMI_$TXn$1_CEC
 $Comp
-L VCC3V3 #PWR06
+L VCC3V3 #PWR110
 U 1 1 57B82B49
 P 10600 4450
-F 0 "#PWR06" H 10600 4300 60  0001 C CNN
+F 0 "#PWR110" H 10600 4300 60  0001 C CNN
 F 1 "VCC3V3" H 10600 4590 60  0000 C CNN
 F 2 "" H 10600 4450 60  0000 C CNN
@@
 $EndComp
 $Comp
-L GND #PWR07
+L GND #PWR109
 U 1 1 57C07776
 P 8550 7150
-F 0 "#PWR07" H 8550 6900 60  0001 C CNN
+F 0 "#PWR109" H 8550 6900 60  0001 C CNN
 F 1 "GND" H 8550 7000 60  0000 C CNN
 F 2 "" H 8550 7150 60  0000 C CNN
@@
 $EndComp
 $Comp
-L VCC3V3 #PWR08
+L VCC3V3 #PWR107
 U 1 1 57B869C2
 P 8400 3600
-F 0 "#PWR08" H 8400 3450 60  0001 C CNN
+F 0 "#PWR107" H 8400 3450 60  0001 C CNN
 F 1 "VCC3V3" H 8400 3740 60  0000 C CNN
 F 2 "" H 8400 3600 60  0000 C CNN
@@
 	8500 4100 8500 4000
 $Comp
-L GND #PWR09
+L GND #PWR108
 U 1 1 57C0777E
 P 8400 4150
-F 0 "#PWR09" H 8400 3900 60  0001 C CNN
+F 0 "#PWR108" H 8400 3900 60  0001 C CNN
 F 1 "GND" H 8400 4000 60  0000 C CNN
 F 2 "" H 8400 4150 60  0000 C CNN
@@
 HDMI_$TXn$1_SDA
 $Comp
-L VCC3V3 #PWR010
+L VCC3V3 #PWR102
 U 1 1 57BC61BF
 P 3100 7110
-F 0 "#PWR010" H 3100 6960 60  0001 C CNN
+F 0 "#PWR102" H 3100 6960 60  0001 C CNN
 F 1 "VCC3V3" H 3315 7165 60  0000 C CNN
 F 2 "" H 3100 7110 60  0000 C CNN
@@
 $EndComp
 $Comp
-L GND #PWR011
+L GND #PWR101
 U 1 1 57C07784
 P 2610 6970
-F 0 "#PWR011" H 2610 6720 60  0001 C CNN
+F 0 "#PWR101" H 2610 6720 60  0001 C CNN
 F 1 "GND" H 2610 6820 60  0000 C CNN
 F 2 "" H 2610 6970 60  0000 C CNN
@@
 	0    1    1    0
 $EndComp
+$Comp
+L ΜA78L00 U$TXn$101
+U 1 1 57E8C5A1
+P 11700 8100
+F 0 "U$TXn$101" H 12000 7800 60  0000 C CNN
+F 1 "ΜA78L00" H 11550 8350 60  0000 C CNN
+F 2 "" H 11700 8100 60  0000 C CNN
+F 3 "" H 11700 8100 60  0000 C CNN
+	1    11700 8100
+	1    0    0    -1
+$EndComp
+$Comp
+L C C$TXn$109
+U 1 1 57E8C7B4
+P 10700 8400
+F 0 "C$TXn$109" H 10725 8500 50  0000 L CNN
+F 1 "0.33uF" H 10725 8300 50  0000 L CNN
+F 2 "" H 10738 8250 50  0000 C CNN
+F 3 "" H 10700 8400 50  0000 C CNN
+	1    10700 8400
+	1    0    0    -1
+$EndComp
+$Comp
+L C C$TXn$110
+U 1 1 57E8C84C
+P 12450 8400
+F 0 "C$TXn$110" H 12475 8500 50  0000 L CNN
+F 1 "0.1uF" H 12475 8300 50  0000 L CNN
+F 2 "" H 12488 8250 50  0000 C CNN
+F 3 "" H 12450 8400 50  0000 C CNN
+	1    12450 8400
+	1    0    0    -1
+$EndComp
+$Comp
+L C C$TXn$111
+U 1 1 57E8C9BD
+P 12800 8400
+F 0 "C$TXn$111" H 12825 8500 50  0000 L CNN
+F 1 "0.1uF" H 12825 8300 50  0000 L CNN
+F 2 "" H 12838 8250 50  0000 C CNN
+F 3 "" H 12800 8400 50  0000 C CNN
+	1    12800 8400
+	1    0    0    -1
+$EndComp
+$Comp
+L R R$TXn$106
+U 1 1 57E8CA09
+P 13100 8400
+F 0 "R$TXn$106" V 13180 8400 50  0000 C CNN
+F 1 "100K" V 13100 8400 50  0000 C CNN
+F 2 "" V 13030 8400 50  0000 C CNN
+F 3 "" H 13100 8400 50  0000 C CNN
+	1    13100 8400
+	1    0    0    -1
+$EndComp
+Wire Wire Line
+	10700 8250 10700 8100
+Wire Wire Line
+	10350 8100 11050 8100
+Wire Wire Line
+	12350 8100 13850 8100
+Wire Wire Line
+	12450 8100 12450 8250
+Wire Wire Line
+	12800 8100 12800 8250
+Connection ~ 12450 8100
+Wire Wire Line
+	13100 8100 13100 8250
+Connection ~ 12800 8100
+Wire Wire Line
+	10700 8550 10700 8700
+Wire Wire Line
+	10700 8700 13100 8700
+Wire Wire Line
+	11700 8650 11700 8750
+Wire Wire Line
+	12450 8700 12450 8550
+Connection ~ 11700 8700
+Wire Wire Line
+	12800 8700 12800 8550
+Connection ~ 12450 8700
+Wire Wire Line
+	13100 8700 13100 8550
+Connection ~ 12800 8700
+Text Label 10700 8100 0    60   ~ 0
+VCC12V0
+Connection ~ 10700 8100
+Text GLabel 10350 8100 0    60   Input ~ 0
+VCC12V0
+Connection ~ 13100 8100
+Text Label 13850 8100 2    60   ~ 0
+$TXn$15V0
+$Comp
+L GND #PWR113
+U 1 1 57E8D9CD
+P 11700 8750
+F 0 "#PWR113" H 11700 8500 60  0001 C CNN
+F 1 "GND" H 11700 8600 60  0000 C CNN
+F 2 "" H 11700 8750 60  0000 C CNN
+F 3 "" H 11700 8750 60  0000 C CNN
+	1    11700 8750
+	1    0    0    -1
+$EndComp
+Text Label 11700 8700 0    60   ~ 0
+GND
+Text GLabel 10300 7650 0    60   Input ~ 0
+VCC3V3
+$Comp
+L VCC3V3 #PWR111
+U 1 1 57E9181D
+P 10650 7600
+F 0 "#PWR111" H 10650 7450 60  0001 C CNN
+F 1 "VCC3V3" H 10650 7740 60  0000 C CNN
+F 2 "" H 10650 7600 60  0000 C CNN
+F 3 "" H 10650 7600 60  0000 C CNN
+	1    10650 7600
+	1    0    0    -1
+$EndComp
+Wire Wire Line
+	10300 7650 10650 7650
+Wire Wire Line
+	10650 7650 10650 7600
+Text Label 10650 7650 2    60   ~ 0
+VCC3V3
 $EndSCHEMATC

Commit message: Change TX template to use a bus like the RX template.
Connections:
- net labels added: HDMI_$TXn$1_D[4..1]
- wire segments 123 -> 131
Changed lines of the file:
@@
 LIBS:hdmi2usb
 LIBS:HDMI2USB-cache
-LIBS:hdmi_TXn-cache
 EELAYER 25 0
 EELAYER END
@@
 Text HLabel 5850 4600 0    60   Input ~ 0
 HDMI_$TXn$1_DDC_EN
-Text HLabel 5400 4800 0    60   Input ~ 0
-HDMI_$TXn$1_D1+
-Text HLabel 5400 4900 0    60   Input ~ 0
-HDMI_$TXn$1_D1-
-Text HLabel 5400 5100 0    60   Input ~ 0
-HDMI_$TXn$1_D2+
-Text HLabel 5400 5200 0    60   Input ~ 0
-HDMI_$TXn$1_D2-
-Text HLabel 5400 5400 0    60   Input ~ 0
-HDMI_$TXn$1_D3+
-Text HLabel 5400 5500 0    60   Input ~ 0
-HDMI_$TXn$1_D3-
-Text HLabel 5400 5700 0    60   Input ~ 0
-HDMI_$TXn$1_D4+
-Text HLabel 5400 5800 0    60   Input ~ 0
-HDMI_$TXn$1_D4-
 Text HLabel 5850 6000 0    60   BiDi ~ 0
 HDMI_$TXn$1_SCL
@@
 Text Label 10650 7650 2    60   ~ 0
 VCC3V3
+Text Label 2650 4950 2    60   ~ 0
+HDMI_$TXn$1_D1+
+Text Label 2650 5050 2    60   ~ 0
+HDMI_$TXn$1_D1-
+Text Label 2650 5250 2    60   ~ 0
+HDMI_$TXn$1_D2+
+Text Label 2650 5350 2    60   ~ 0
+HDMI_$TXn$1_D2-
+Text Label 2650 5550 2    60   ~ 0
+HDMI_$TXn$1_D3+
+Text Label 2650 5650 2    60   ~ 0
+HDMI_$TXn$1_D3-
+Text Label 2650 5850 2    60   ~ 0
+HDMI_$TXn$1_D4+
+Text Label 2650 5950 2    60   ~ 0
+HDMI_$TXn$1_D4-
+Wire Wire Line
+	1850 5850 2650 5850
+Wire Wire Line
+	1850 5950 2650 5950
+Wire Wire Line
+	1850 5650 2650 5650
+Wire Wire Line
+	1850 5550 2650 5550
+Wire Wire Line
+	1850 5350 2650 5350
+Wire Wire Line
+	1850 5250 2650 5250
+Wire Wire Line
+	1850 5050 2650 5050
+Wire Wire Line
+	1850 4950 2650 4950
+Text HLabel 1550 4825 0    60   Input ~ 0
+HDMI_$TXn$1_D[4..1]
+Entry Wire Line
+	1750 4850 1850 4950
+Entry Wire Line
+	1750 4950 1850 5050
+Entry Wire Line
+	1750 5150 1850 5250
+Entry Wire Line
+	1750 5250 1850 5350
+Entry Wire Line
+	1750 5450 1850 5550
+Entry Wire Line
+	1750 5550 1850 5650
+Entry Wire Line
+	1750 5750 1850 5850
+Entry Wire Line
+	1750 5850 1850 5950
+Wire Bus Line
+	1750 5850 1750 4825
+Wire Bus Line
+	1750 4825 1550 4825
 $EndSCHEMATC

Commit message: Revert "Change TX template to use a bus like the RX template."
This reverts commit be1a1c4228a1cc4095e9d422f81658321b378f5c.
Connections:
- net labels removed: HDMI_$TXn$1_D[4..1]
- wire segments 131 -> 123
Changed lines of the file:
@@
 LIBS:hdmi2usb
 LIBS:HDMI2USB-cache
+LIBS:hdmi_TXn-cache
 EELAYER 25 0
 EELAYER END
@@
 Text HLabel 5850 4600 0    60   Input ~ 0
 HDMI_$TXn$1_DDC_EN
+Text HLabel 5400 4800 0    60   Input ~ 0
+HDMI_$TXn$1_D1+
+Text HLabel 5400 4900 0    60   Input ~ 0
+HDMI_$TXn$1_D1-
+Text HLabel 5400 5100 0    60   Input ~ 0
+HDMI_$TXn$1_D2+
+Text HLabel 5400 5200 0    60   Input ~ 0
+HDMI_$TXn$1_D2-
+Text HLabel 5400 5400 0    60   Input ~ 0
+HDMI_$TXn$1_D3+
+Text HLabel 5400 5500 0    60   Input ~ 0
+HDMI_$TXn$1_D3-
+Text HLabel 5400 5700 0    60   Input ~ 0
+HDMI_$TXn$1_D4+
+Text HLabel 5400 5800 0    60   Input ~ 0
+HDMI_$TXn$1_D4-
 Text HLabel 5850 6000 0    60   BiDi ~ 0
 HDMI_$TXn$1_SCL
@@
 Text Label 10650 7650 2    60   ~ 0
 VCC3V3
-Text Label 2650 4950 2    60   ~ 0
-HDMI_$TXn$1_D1+
-Text Label 2650 5050 2    60   ~ 0
-HDMI_$TXn$1_D1-
-Text Label 2650 5250 2    60   ~ 0
-HDMI_$TXn$1_D2+
-Text Label 2650 5350 2    60   ~ 0
-HDMI_$TXn$1_D2-
-Text Label 2650 5550 2    60   ~ 0
-HDMI_$TXn$1_D3+
-Text Label 2650 5650 2    60   ~ 0
-HDMI_$TXn$1_D3-
-Text Label 2650 5850 2    60   ~ 0
-HDMI_$TXn$1_D4+
-Text Label 2650 5950 2    60   ~ 0
-HDMI_$TXn$1_D4-
-Wire Wire Line
-	1850 5850 2650 5850
-Wire Wire Line
-	1850 5950 2650 5950
-Wire Wire Line
-	1850 5650 2650 5650
-Wire Wire Line
-	1850 5550 2650 5550
-Wire Wire Line
-	1850 5350 2650 5350
-Wire Wire Line
-	1850 5250 2650 5250
-Wire Wire Line
-	1850 5050 2650 5050
-Wire Wire Line
-	1850 4950 2650 4950
-Text HLabel 1550 4825 0    60   Input ~ 0
-HDMI_$TXn$1_D[4..1]
-Entry Wire Line
-	1750 4850 1850 4950
-Entry Wire Line
-	1750 4950 1850 5050
-Entry Wire Line
-	1750 5150 1850 5250
-Entry Wire Line
-	1750 5250 1850 5350
-Entry Wire Line
-	1750 5450 1850 5550
-Entry Wire Line
-	1750 5550 1850 5650
-Entry Wire Line
-	1750 5750 1850 5850
-Entry Wire Line
-	1750 5850 1850 5950
-Wire Bus Line
-	1750 5850 1750 4825
-Wire Bus Line
-	1750 4825 1550 4825
 $EndSCHEMATC
