File: DDRn.sch (KiCad schematic (older format))
At the start: 56 parts

Commit message: Fixing the DDR component name.
Parts:
- renumbered U$DDRn$1 to U$DDRn$
Changed lines of the file:
@@
 $EndDescr
 $Comp
-L MT41J128M16 U$DDRn$1
+L MT41J128M16 U$DDRn$
 U 1 1 57C61740
 P 8400 5050
-F 0 "U$DDRn$1" H 8350 7900 60  0000 C CNN
+F 0 "U$DDRn$" H 8350 7900 60  0000 C CNN
 F 1 "MT41J128M16" H 8350 1500 60  0000 C CNN
 F 2 "~" H 8400 5050 60  0000 C CNN

Commit message: Adding footprints to DDR template.
Parts:
- C$DDRn$1, C$DDRn$10, C$DDRn$11, C$DDRn$12, C$DDRn$13, C$DDRn$14, C$DDRn$15, C$DDRn$16, C$DDRn$17, C$DDRn$18, C$DDRn$19, C$DDRn$2, C$DDRn$20, C$DDRn$21, C$DDRn$22, C$DDRn$23, C$DDRn$24, C$DDRn$25, C$DDRn$26, C$DDRn$27, C$DDRn$28, C$DDRn$29, C$DDRn$3, C$DDRn$30, C$DDRn$31, C$DDRn$32, C$DDRn$33, C$DDRn$34, C$DDRn$35, C$DDRn$36, C$DDRn$37, C$DDRn$38, C$DDRn$39, C$DDRn$4, C$DDRn$40, C$DDRn$41, C$DDRn$42, C$DDRn$43, C$DDRn$5, C$DDRn$6, C$DDRn$7, C$DDRn$8, C$DDRn$9: footprint (none) -> Capacitors_SMD:C_0402
- R$DDRn$1, R$DDRn$11, R$DDRn$12, R$DDRn$4, R$DDRn$5, R$DDRn$6, R$DDRn$8: footprint (none) -> Resistors_SMD:R_0402
- R$DDRn$10, R$DDRn$2, R$DDRn$3, R$DDRn$7, R$DDRn$9: footprint ~ -> Resistors_SMD:R_Array_Concave_4x0402
- U$DDRn$0: renamed from U$DDRn$; footprint ~ -> SMD_Packages:BGA-96_pitch0.8mm_dia0.4mm; desc (none) -> DDR3 SDRAM 2GBIT 800MHz; manf# (none) -> MT41J128M16JT-125
Connections:
- wire segments 362 -> 218

Commit message: Make sure all values have a leading zero.
Parts:
- renumbered C$DDRn$1 to C$DDRn$01, C$DDRn$2 to C$DDRn$02, C$DDRn$3 to C$DDRn$03, C$DDRn$4 to C$DDRn$04, C$DDRn$5 to C$DDRn$05, C$DDRn$6 to C$DDRn$06, C$DDRn$7 to C$DDRn$07, C$DDRn$8 to C$DDRn$08, C$DDRn$9 to C$DDRn$09, R$DDRn$1 to R$DDRn$01, R$DDRn$2 to R$DDRn$02, R$DDRn$3 to R$DDRn$03, R$DDRn$4 to R$DDRn$04, R$DDRn$5 to R$DDRn$05, R$DDRn$6 to R$DDRn$06, R$DDRn$7 to R$DDRn$07, R$DDRn$8 to R$DDRn$08, R$DDRn$9 to R$DDRn$09
Changed lines of the file:
@@
 $EndComp
 $Comp
-L R R$DDRn$1
+L R R$DDRn$01
 U 1 1 57C61743
 P 2500 10550
-F 0 "R$DDRn$1" V 2580 10550 50  0000 C CNN
+F 0 "R$DDRn$01" V 2580 10550 50  0000 C CNN
 F 1 "R" V 2500 10550 50  0000 C CNN
 F 2 "Resistors_SMD:R_0402" H 2500 10550 60  0001 C CNN
@@
 $EndComp
 $Comp
-L RES_NET4 R$DDRn$9
+L RES_NET4 R$DDRn$09
 U 1 1 57C61745
 P 5595 10535
-F 0 "R$DDRn$9" H 5595 10285 60  0000 C CNN
+F 0 "R$DDRn$09" H 5595 10285 60  0000 C CNN
 F 1 "49.9E" H 5595 10885 60  0000 C CNN
 F 2 "Resistors_SMD:R_Array_Concave_4x0402" H 5595 10535 60  0001 C CNN
@@
 $EndComp
 $Comp
-L RES_NET4 R$DDRn$7
+L RES_NET4 R$DDRn$07
 U 1 1 57C61746
 P 4745 10535
-F 0 "R$DDRn$7" H 4745 10285 60  0000 C CNN
+F 0 "R$DDRn$07" H 4745 10285 60  0000 C CNN
 F 1 "49.9E" H 4745 10885 60  0000 C CNN
 F 2 "Resistors_SMD:R_Array_Concave_4x0402" H 4745 10535 60  0001 C CNN
@@
 $EndComp
 $Comp
-L RES_NET4 R$DDRn$3
+L RES_NET4 R$DDRn$03
 U 1 1 57C61747
 P 3895 10535
-F 0 "R$DDRn$3" H 3895 10285 60  0000 C CNN
+F 0 "R$DDRn$03" H 3895 10285 60  0000 C CNN
 F 1 "49.9E" H 3895 10885 60  0000 C CNN
 F 2 "Resistors_SMD:R_Array_Concave_4x0402" H 3895 10535 60  0001 C CNN
@@
 $EndComp
 $Comp
-L RES_NET4 R$DDRn$2
+L RES_NET4 R$DDRn$02
 U 1 1 57C61748
 P 3045 10535
-F 0 "R$DDRn$2" H 3045 10285 60  0000 C CNN
+F 0 "R$DDRn$02" H 3045 10285 60  0000 C CNN
 F 1 "49.9E" H 3045 10885 60  0000 C CNN
 F 2 "Resistors_SMD:R_Array_Concave_4x0402" H 3045 10535 60  0001 C CNN
@@
 $EndComp
 $Comp
-L R R$DDRn$4
+L R R$DDRn$04
 U 1 1 57C6174E
 P 4300 4750
-F 0 "R$DDRn$4" V 4350 4550 50  0000 C CNN
+F 0 "R$DDRn$04" V 4350 4550 50  0000 C CNN
 F 1 "100E" V 4300 4750 50  0000 C CNN
 F 2 "Resistors_SMD:R_0402" H 4300 4750 60  0001 C CNN
@@
 $EndComp
 $Comp
-L R R$DDRn$8
+L R R$DDRn$08
 U 1 1 57C6174F
 P 4850 6400
-F 0 "R$DDRn$8" V 4930 6400 50  0000 C CNN
+F 0 "R$DDRn$08" V 4930 6400 50  0000 C CNN
 F 1 "4K7" V 4850 6400 50  0000 C CNN
 F 2 "Resistors_SMD:R_0402" H 4850 6400 60  0001 C CNN
@@
 $EndComp
 $Comp
-L R R$DDRn$6
+L R R$DDRn$06
 U 1 1 57C61750
 P 4600 6400
-F 0 "R$DDRn$6" V 4680 6400 50  0000 C CNN
+F 0 "R$DDRn$06" V 4680 6400 50  0000 C CNN
 F 1 "4K7" V 4600 6400 50  0000 C CNN
 F 2 "Resistors_SMD:R_0402" H 4600 6400 60  0001 C CNN
@@
 $EndComp
 $Comp
-L R R$DDRn$5
+L R R$DDRn$05
 U 1 1 57C61752
 P 4350 6400
-F 0 "R$DDRn$5" V 4430 6400 50  0000 C CNN
+F 0 "R$DDRn$05" V 4430 6400 50  0000 C CNN
 F 1 "4K7" V 4350 6400 50  0000 C CNN
 F 2 "Resistors_SMD:R_0402" H 4350 6400 60  0001 C CNN
@@
 $EndComp
 $Comp
-L C C$DDRn$3
+L C C$DDRn$03
 U 1 1 57C61753
 P 2250 13650
-F 0 "C$DDRn$3" H 2300 13750 50  0000 L CNN
+F 0 "C$DDRn$03" H 2300 13750 50  0000 L CNN
 F 1 "0.1uF" H 2300 13550 50  0000 L CNN
 F 2 "Capacitors_SMD:C_0402" H 2250 13650 60  0001 C CNN
@@
 $EndComp
 $Comp
-L C C$DDRn$6
+L C C$DDRn$06
 U 1 1 57C61754
 P 2600 13650
-F 0 "C$DDRn$6" H 2650 13750 50  0000 L CNN
+F 0 "C$DDRn$06" H 2650 13750 50  0000 L CNN
 F 1 "0.1uF" H 2650 13550 50  0000 L CNN
 F 2 "Capacitors_SMD:C_0402" H 2600 13650 60  0001 C CNN
@@
 $EndComp
 $Comp
-L C C$DDRn$9
+L C C$DDRn$09
 U 1 1 57C61755
 P 3000 13650
-F 0 "C$DDRn$9" H 3050 13750 50  0000 L CNN
+F 0 "C$DDRn$09" H 3050 13750 50  0000 L CNN
 F 1 "0.1uF" H 3050 13550 50  0000 L CNN
 F 2 "Capacitors_SMD:C_0402" H 3000 13650 60  0001 C CNN
@@
 $EndComp
 $Comp
-L C C$DDRn$2
+L C C$DDRn$02
 U 1 1 57C61762
 P 2250 13150
-F 0 "C$DDRn$2" H 2300 13250 50  0000 L CNN
+F 0 "C$DDRn$02" H 2300 13250 50  0000 L CNN
 F 1 "0.1uF" H 2300 13050 50  0000 L CNN
 F 2 "Capacitors_SMD:C_0402" H 2250 13150 60  0001 C CNN
@@
 $EndComp
 $Comp
-L C C$DDRn$5
+L C C$DDRn$05
 U 1 1 57C61763
 P 2600 13150
-F 0 "C$DDRn$5" H 2650 13250 50  0000 L CNN
+F 0 "C$DDRn$05" H 2650 13250 50  0000 L CNN
 F 1 "0.1uF" H 2650 13050 50  0000 L CNN
 F 2 "Capacitors_SMD:C_0402" H 2600 13150 60  0001 C CNN
@@
 $EndComp
 $Comp
-L C C$DDRn$8
+L C C$DDRn$08
 U 1 1 57C61764
 P 3000 13150
-F 0 "C$DDRn$8" H 3050 13250 50  0000 L CNN
+F 0 "C$DDRn$08" H 3050 13250 50  0000 L CNN
 F 1 "0.1uF" H 3050 13050 50  0000 L CNN
 F 2 "Capacitors_SMD:C_0402" H 3000 13150 60  0001 C CNN
@@
 VTTREF0
 $Comp
-L C C$DDRn$1
+L C C$DDRn$01
 U 1 1 57C617AD
 P 2230 14695
-F 0 "C$DDRn$1" H 2280 14795 50  0000 L CNN
+F 0 "C$DDRn$01" H 2280 14795 50  0000 L CNN
 F 1 "0.1uF" H 2280 14595 50  0000 L CNN
 F 2 "Capacitors_SMD:C_0402" H 2230 14695 60  0001 C CNN
@@
 $EndComp
 $Comp
-L C C$DDRn$4
+L C C$DDRn$04
 U 1 1 57C617AE
 P 2530 14695
-F 0 "C$DDRn$4" H 2580 14795 50  0000 L CNN
+F 0 "C$DDRn$04" H 2580 14795 50  0000 L CNN
 F 1 "0.1uF" H 2580 14595 50  0000 L CNN
 F 2 "Capacitors_SMD:C_0402" H 2530 14695 60  0001 C CNN
@@
 $EndComp
 $Comp
-L C C$DDRn$7
+L C C$DDRn$07
 U 1 1 57C617AF
 P 2830 14695
-F 0 "C$DDRn$7" H 2880 14795 50  0000 L CNN
+F 0 "C$DDRn$07" H 2880 14795 50  0000 L CNN
 F 1 "0.1uF" H 2880 14595 50  0000 L CNN
 F 2 "Capacitors_SMD:C_0402" H 2830 14695 60  0001 C CNN

Commit message: Capacitors are actually 0402 parts.
Parts:
- C$DDRn$01, C$DDRn$02, C$DDRn$03, C$DDRn$04, C$DDRn$05, C$DDRn$06, C$DDRn$07, C$DDRn$08, C$DDRn$09, C$DDRn$10, C$DDRn$11, C$DDRn$12, C$DDRn$13, C$DDRn$14, C$DDRn$15, C$DDRn$16, C$DDRn$17, C$DDRn$18, C$DDRn$19, C$DDRn$20, C$DDRn$21, C$DDRn$22, C$DDRn$23, C$DDRn$24, C$DDRn$25, C$DDRn$26, C$DDRn$27, C$DDRn$28, C$DDRn$29, C$DDRn$30, C$DDRn$31, C$DDRn$32, C$DDRn$33, C$DDRn$34, C$DDRn$35, C$DDRn$36, C$DDRn$37, C$DDRn$38, C$DDRn$39, C$DDRn$40, C$DDRn$41, C$DDRn$42, C$DDRn$43: footprint Capacitors_SMD:C_0402 -> Capacitors_SMD:C_0201
- R$DDRn$01: footprint Resistors_SMD:R_0402 -> Resistors_SMD:R_0603

Commit message: Always have a prefix 1.
Parts:
- renumbered C$DDRn$01 to C$DDRn$101, C$DDRn$02 to C$DDRn$102, C$DDRn$03 to C$DDRn$103, C$DDRn$04 to C$DDRn$104, C$DDRn$05 to C$DDRn$105, C$DDRn$06 to C$DDRn$106, C$DDRn$07 to C$DDRn$107, C$DDRn$08 to C$DDRn$108, C$DDRn$09 to C$DDRn$109, C$DDRn$10 to C$DDRn$110, C$DDRn$11 to C$DDRn$111, C$DDRn$12 to C$DDRn$112, C$DDRn$13 to C$DDRn$113, C$DDRn$14 to C$DDRn$114, C$DDRn$15 to C$DDRn$115, C$DDRn$16 to C$DDRn$116, C$DDRn$17 to C$DDRn$117, C$DDRn$18 to C$DDRn$118, C$DDRn$19 to C$DDRn$119, C$DDRn$20 to C$DDRn$120, C$DDRn$21 to C$DDRn$121, C$DDRn$22 to C$DDRn$122, C$DDRn$23 to C$DDRn$123, C$DDRn$24 to C$DDRn$124, C$DDRn$25 to C$DDRn$125, C$DDRn$26 to C$DDRn$126, C$DDRn$27 to C$DDRn$127, C$DDRn$28 to C$DDRn$128, C$DDRn$29 to C$DDRn$129, C$DDRn$30 to C$DDRn$130, C$DDRn$31 to C$DDRn$131, C$DDRn$32 to C$DDRn$132, C$DDRn$33 to C$DDRn$133, C$DDRn$34 to C$DDRn$134, C$DDRn$35 to C$DDRn$135, C$DDRn$36 to C$DDRn$136, C$DDRn$37 to C$DDRn$137, C$DDRn$38 to C$DDRn$138, C$DDRn$39 to C$DDRn$139, C$DDRn$40 to C$DDRn$140, C$DDRn$41 to C$DDRn$141, C$DDRn$42 to C$DDRn$142, C$DDRn$43 to C$DDRn$143, R$DDRn$01 to R$DDRn$101, R$DDRn$02 to R$DDRn$102, R$DDRn$03 to R$DDRn$103, R$DDRn$04 to R$DDRn$104, R$DDRn$05 to R$DDRn$105, R$DDRn$06 to R$DDRn$106, R$DDRn$07 to R$DDRn$107, R$DDRn$08 to R$DDRn$108, R$DDRn$09 to R$DDRn$109, R$DDRn$10 to R$DDRn$110, R$DDRn$11 to R$DDRn$111, R$DDRn$12 to R$DDRn$112, U$DDRn$0 to U$DDRn$10
Connections:
- net labels added: $DDRn$1_A0, $DDRn$1_A1, $DDRn$1_A10, $DDRn$1_A11, $DDRn$1_A12, $DDRn$1_A13, $DDRn$1_A14, $DDRn$1_A2, $DDRn$1_A3, $DDRn$1_A4, $DDRn$1_A5, $DDRn$1_A6, $DDRn$1_A7, $DDRn$1_A8, $DDRn$1_A9, $DDRn$1_A[0..14], $DDRn$1_BA0, $DDRn$1_BA1, $DDRn$1_BA2, $DDRn$1_BA[0..2], $DDRn$1_CASN0, $DDRn$1_CAS_N, $DDRn$1_CKE, $DDRn$1_CK_N, $DDRn$1_CK_P, $DDRn$1_CS_N, $DDRn$1_DQ0, $DDRn$1_DQ1, $DDRn$1_DQ10, $DDRn$1_DQ11, $DDRn$1_DQ12, $DDRn$1_DQ13, $DDRn$1_DQ14, $DDRn$1_DQ15, $DDRn$1_DQ2, $DDRn$1_DQ3, $DDRn$1_DQ4, $DDRn$1_DQ5, $DDRn$1_DQ6, $DDRn$1_DQ7, $DDRn$1_DQ8, $DDRn$1_DQ9, $DDRn$1_DQ[0..15], $DDRn$1_LDM, $DDRn$1_LDQS_N, $DDRn$1_LDQS_P, $DDRn$1_ODT, $DDRn$1_RASN0, $DDRn$1_RAS_N, $DDRn$1_RESET_N, $DDRn$1_UDM, $DDRn$1_UDQS_N, $DDRn$1_UDQS_P, $DDRn$1_WE0, $DDRn$1_WE_N, $DDRn$1_ZQ, VTT$DDRn$1
- net labels removed: $DDRn$_A0, $DDRn$_A1, $DDRn$_A10, $DDRn$_A11, $DDRn$_A12, $DDRn$_A13, $DDRn$_A14, $DDRn$_A2, $DDRn$_A3, $DDRn$_A4, $DDRn$_A5, $DDRn$_A6, $DDRn$_A7, $DDRn$_A8, $DDRn$_A9, $DDRn$_A[0..14], $DDRn$_BA0, $DDRn$_BA1, $DDRn$_BA2, $DDRn$_BA[0..2], $DDRn$_CASN0, $DDRn$_CAS_N, $DDRn$_CKE, $DDRn$_CK_N, $DDRn$_CK_P, $DDRn$_CS_N, $DDRn$_DQ0, $DDRn$_DQ1, $DDRn$_DQ10, $DDRn$_DQ11, $DDRn$_DQ12, $DDRn$_DQ13, $DDRn$_DQ14, $DDRn$_DQ15, $DDRn$_DQ2, $DDRn$_DQ3, $DDRn$_DQ4, $DDRn$_DQ5, $DDRn$_DQ6, $DDRn$_DQ7, $DDRn$_DQ8, $DDRn$_DQ9, $DDRn$_DQ[0..15], $DDRn$_LDM, $DDRn$_LDQS_N, $DDRn$_LDQS_P, $DDRn$_ODT, $DDRn$_RASN0, $DDRn$_RAS_N, $DDRn$_RESET_N, $DDRn$_UDM, $DDRn$_UDQS_N, $DDRn$_UDQS_P, $DDRn$_WE0, $DDRn$_WE_N, $DDRn$_ZQ, VTT$DDRn$

Commit message: Small fixes to major component numbers.
Parts:
- renumbered U$DDRn$10 to U$DDRn$1
Changed lines of the file:
@@
 $EndDescr
 $Comp
-L MT41J128M16 U$DDRn$10
+L MT41J128M16 U$DDRn$1
 U 1 1 57C61740
 P 8400 5050
-F 0 "U$DDRn$10" H 8350 7900 60  0000 C CNN
+F 0 "U$DDRn$1" H 8350 7900 60  0000 C CNN
 F 1 "MT41J128M16" H 8350 1500 60  0000 C CNN
 F 2 "SMD_Packages:BGA-96_pitch0.8mm_dia0.4mm" H 8400 5050 60  0001 C CNN

Commit message: Updating labels and getting VTT right.
Connections:
- net labels added: VTTDDR, VTTREF
- net labels removed: VTT$DDRn$1, VTTREF0
Changed lines of the file:
@@
 $EndComp
 Text Label 2095 10235 0    60   ~ 0
-VTT$DDRn$1
+VTTDDR
 $Comp
 L R R$DDRn$111
@@
 VCC1V5
 Text Label 1800 13950 0    60   ~ 0
-VTT$DDRn$1
+VTTDDR
 Text Label 2400 2450 0    60   ~ 12
 $DDRn$1_A0
@@
 VCC1V5
 Text GLabel 1695 10235 0    60   Input ~ 12
-VTT$DDRn$1
+VTTDDR
 Text HLabel 9350 2250 2    60   Input ~ 12
 $DDRn$1_ZQ
 Text GLabel 9350 4650 2    60   Input ~ 0
-VTTREF0
+VTTREF
 $Comp
 L C C$DDRn$101
@@
 $EndComp
 Text Label 5030 14995 0    60   ~ 0
-VTT$DDRn$1
+VTTDDR
 $Comp
 L GND #PWR07
@@
 Connection ~ 9250 3900
 Wire Wire Line
-	9200 4000 9250 4000
+	9200 4000 9510 4000
 Connection ~ 9250 4000
 Wire Wire Line
@@
 Connection ~ 9250 2950
 Wire Wire Line
-	9200 3050 9250 3050
+	9200 3050 9510 3050
 Connection ~ 9250 3050
 Wire Wire Line
@@
 	2230 14990 2530 14995
 Wire Wire Line
-	2530 14995 5030 14995
+	2530 14995 5505 14995
 Wire Wire Line
 	4980 14845 4980 14995
@@
 Text Notes 11780 2715 0    197  ~ 39
 $WARNING1$\n$WARNING2$\n$WARNING3$
+Text GLabel 1800 13950 0    60   Input ~ 12
+VTTDDR
+Text GLabel 5505 14995 2    60   Input ~ 12
+VTTDDR
+Text GLabel 9510 3050 2    60   Input ~ 12
+VCC1V5
+Text GLabel 9510 4000 2    60   Input ~ 12
+VCC1V5
 $EndSCHEMATC

Commit message: Remove external terminations and associated connections. Add `Vref` connections as per arty/nexys-video/neso
Parts:
- removed C$DDRn$101, C$DDRn$103, C$DDRn$104, C$DDRn$106, C$DDRn$107, C$DDRn$109, C$DDRn$110, C$DDRn$112, C$DDRn$113, C$DDRn$114, C$DDRn$116, C$DDRn$117, C$DDRn$119, C$DDRn$120, C$DDRn$122, C$DDRn$123, C$DDRn$125, C$DDRn$126, C$DDRn$128, C$DDRn$130, C$DDRn$132, C$DDRn$134, C$DDRn$136, C$DDRn$138, C$DDRn$140: 0.1uF, Capacitors_SMD:C_0201, symbol C
- removed R$DDRn$101: R, Resistors_SMD:R_0603, symbol R
- removed R$DDRn$102, R$DDRn$103, R$DDRn$107, R$DDRn$109, R$DDRn$110: 49.9E, Resistors_SMD:R_Array_Concave_4x0402, symbol RES_NET4
- added C$DDRn$? (x4): 0.1uF, Capacitors_SMD:C_0402, symbol C
- added C$DDRn$? (x2): 10nF, Capacitors_SMD:C_0402, symbol C
- C$DDRn$102, C$DDRn$105, C$DDRn$108, C$DDRn$111, C$DDRn$115, C$DDRn$118, C$DDRn$121, C$DDRn$124, C$DDRn$127, C$DDRn$129, C$DDRn$131, C$DDRn$133, C$DDRn$135, C$DDRn$137, C$DDRn$139, C$DDRn$141, C$DDRn$142: footprint Capacitors_SMD:C_0201 -> Capacitors_SMD:C_0402
- C$DDRn$143: value 0.1uF -> 1uF; footprint Capacitors_SMD:C_0201 -> Capacitors_SMD:C_0402
- R$DDRn$112: value R -> 240R
Connections:
- net labels added: VCC0V75
- net labels removed: $DDRn$1_ZQ, VTTDDR, VTTREF
- wire segments 218 -> 254
Other:
- note added: "CA Bypass"
- note added: "DQ Bypass\n"
