File: DDRn.sch (KiCad schematic (older format))
At the start: 31 parts

Commit message: Move 0.75V power supply to DDR template
Parts:
- added R$DDRn$? (x2): 1K, Resistors_SMD:R_0402, symbol R
Connections:
- wire segments 254 -> 168
Other:
- moved on the sheet: C$DDRn$?

Commit message: Annotate new components in ddr3 template
Parts:
- gave numbers to parts that had none: 8
Connections:
- wire segments 168 -> 261

Commit message: Change 0.75V net from global to local
Connections:
- net labels added: $DDRn$10V75
- net labels removed: VCC0V75
- wire segments 261 -> 260
Changed lines of the file:
@@
 Text GLabel 1800 12850 0    60   Input ~ 12
 VCC1V5
-Text GLabel 11100 4750 2    60   Input ~ 12
-VCC0V75
 Text Label 2250 5650 0    60   ~ 0
 $DDRn$1_CASN0
@@
 	10150 4750 10950 4750
 Wire Wire Line
-	10950 4750 11100 4750
+	10950 4750 11650 4750
 Wire Wire Line
 	9250 4750 9250 4850
@@
 	-1   0    0    1
 $EndComp
-Text GLabel 1800 14150 0    60   Input ~ 12
-VCC0V75
-Wire Wire Line
-	1800 14150 2250 14150
+Wire Wire Line
+	1550 14150 2250 14150
 Wire Wire Line
 	2250 14150 2600 14150
@@
 	10150 4000 10150 4250
 Wire Wire Line
-	8400 13400 8400 13300
+	8400 13300 8400 13550
 $Comp
 L R R$DDRn$102
@@
 Connection ~ 10150 4000
 Connection ~ 10950 4000
-Wire Wire Line
-	8400 13400 8400 13550
 $Comp
 L GND #PWR?
@@
 Text Label 8400 13550 0    60   ~ 0
 GND
+Text Label 11650 4750 2    60   ~ 0
+$DDRn$10V75
+Text Label 1550 14150 0    60   ~ 0
+$DDRn$10V75
 $EndSCHEMATC

Commit message: Fixing up the labels a little.
Connections:
- wire segments 260 -> 261
Other:
- moved on the sheet: C$DDRn$141, C$DDRn$142
Changed lines of the file:
@@
 LIBS:hdmi2usb
 LIBS:HDMI2USB-cache
-LIBS:DDRn-cache
 EELAYER 25 0
 EELAYER END
@@
 U 1 1 57C61762
 P 2250 13150
-F 0 "C$DDRn$102" H 2300 13250 50  0000 L CNN
-F 1 "0.1uF" H 2300 13050 50  0000 L CNN
+F 0 "C$DDRn$102" V 2250 13450 50  0000 L CNN
+F 1 "0.1uF" H 2275 13050 50  0000 L CNN
 F 2 "Capacitors_SMD:C_0402" H 2250 13150 60  0001 C CNN
 F 3 "" H 2250 13150 60  0000 C CNN
@@
 U 1 1 57C61763
 P 2600 13150
-F 0 "C$DDRn$105" H 2650 13250 50  0000 L CNN
-F 1 "0.1uF" H 2650 13050 50  0000 L CNN
+F 0 "C$DDRn$105" V 2600 13450 50  0000 L CNN
+F 1 "0.1uF" H 2625 13050 50  0000 L CNN
 F 2 "Capacitors_SMD:C_0402" H 2600 13150 60  0001 C CNN
 F 3 "" H 2600 13150 60  0000 C CNN
@@
 U 1 1 57C61764
 P 3000 13150
-F 0 "C$DDRn$108" H 3050 13250 50  0000 L CNN
-F 1 "0.1uF" H 3050 13050 50  0000 L CNN
+F 0 "C$DDRn$108" V 3000 13450 50  0000 L CNN
+F 1 "0.1uF" H 3025 13050 50  0000 L CNN
 F 2 "Capacitors_SMD:C_0402" H 3000 13150 60  0001 C CNN
 F 3 "" H 3000 13150 60  0000 C CNN
@@
 U 1 1 57C61765
 P 3400 13150
-F 0 "C$DDRn$111" H 3450 13250 50  0000 L CNN
-F 1 "0.1uF" H 3450 13050 50  0000 L CNN
+F 0 "C$DDRn$111" V 3400 13450 50  0000 L CNN
+F 1 "0.1uF" H 3425 13050 50  0000 L CNN
 F 2 "Capacitors_SMD:C_0402" H 3400 13150 60  0001 C CNN
 F 3 "" H 3400 13150 60  0000 C CNN
@@
 U 1 1 57C61766
 P 3750 13150
-F 0 "C$DDRn$115" H 3800 13250 50  0000 L CNN
-F 1 "0.1uF" H 3800 13050 50  0000 L CNN
+F 0 "C$DDRn$115" V 3750 13450 50  0000 L CNN
+F 1 "0.1uF" H 3775 13050 50  0000 L CNN
 F 2 "Capacitors_SMD:C_0402" H 3750 13150 60  0001 C CNN
 F 3 "" H 3750 13150 60  0000 C CNN
@@
 U 1 1 57C61767
 P 4100 13150
-F 0 "C$DDRn$118" H 4150 13250 50  0000 L CNN
-F 1 "0.1uF" H 4150 13050 50  0000 L CNN
+F 0 "C$DDRn$118" V 4100 13450 50  0000 L CNN
+F 1 "0.1uF" H 4125 13050 50  0000 L CNN
 F 2 "Capacitors_SMD:C_0402" H 4100 13150 60  0001 C CNN
 F 3 "" H 4100 13150 60  0000 C CNN
@@
 U 1 1 57C61768
 P 4550 13150
-F 0 "C$DDRn$121" H 4600 13250 50  0000 L CNN
-F 1 "0.1uF" H 4600 13050 50  0000 L CNN
+F 0 "C$DDRn$121" V 4550 13450 50  0000 L CNN
+F 1 "0.1uF" H 4575 13050 50  0000 L CNN
 F 2 "Capacitors_SMD:C_0402" H 4550 13150 60  0001 C CNN
 F 3 "" H 4550 13150 60  0000 C CNN
@@
 U 1 1 57C61769
 P 4950 13150
-F 0 "C$DDRn$124" H 5000 13250 50  0000 L CNN
-F 1 "0.1uF" H 5000 13050 50  0000 L CNN
+F 0 "C$DDRn$124" V 4950 13450 50  0000 L CNN
+F 1 "0.1uF" H 4975 13050 50  0000 L CNN
 F 2 "Capacitors_SMD:C_0402" H 4950 13150 60  0001 C CNN
 F 3 "" H 4950 13150 60  0000 C CNN
@@
 U 1 1 57C6176A
 P 5350 13150
-F 0 "C$DDRn$127" H 5400 13250 50  0000 L CNN
-F 1 "0.1uF" H 5400 13050 50  0000 L CNN
+F 0 "C$DDRn$127" V 5350 13450 50  0000 L CNN
+F 1 "0.1uF" H 5375 13050 50  0000 L CNN
 F 2 "Capacitors_SMD:C_0402" H 5350 13150 60  0001 C CNN
 F 3 "" H 5350 13150 60  0000 C CNN
@@
 U 1 1 57C6176B
 P 5700 13150
-F 0 "C$DDRn$129" H 5750 13250 50  0000 L CNN
-F 1 "0.1uF" H 5750 13050 50  0000 L CNN
+F 0 "C$DDRn$129" V 5700 13450 50  0000 L CNN
+F 1 "0.1uF" H 5725 13050 50  0000 L CNN
 F 2 "Capacitors_SMD:C_0402" H 5700 13150 60  0001 C CNN
 F 3 "" H 5700 13150 60  0000 C CNN
@@
 U 1 1 57C6176C
 P 6150 13150
-F 0 "C$DDRn$131" H 6200 13250 50  0000 L CNN
-F 1 "0.1uF" H 6200 13050 50  0000 L CNN
+F 0 "C$DDRn$131" V 6150 13450 50  0000 L CNN
+F 1 "0.1uF" H 6175 13050 50  0000 L CNN
 F 2 "Capacitors_SMD:C_0402" H 6150 13150 60  0001 C CNN
 F 3 "" H 6150 13150 60  0000 C CNN
@@
 U 1 1 57C6176D
 P 6600 13150
-F 0 "C$DDRn$133" H 6650 13250 50  0000 L CNN
-F 1 "0.1uF" H 6650 13050 50  0000 L CNN
+F 0 "C$DDRn$133" V 6600 13450 50  0000 L CNN
+F 1 "0.1uF" H 6625 13050 50  0000 L CNN
 F 2 "Capacitors_SMD:C_0402" H 6600 13150 60  0001 C CNN
 F 3 "" H 6600 13150 60  0000 C CNN
@@
 U 1 1 57C6176E
 P 7000 13150
-F 0 "C$DDRn$135" H 7050 13250 50  0000 L CNN
-F 1 "0.1uF" H 7050 13050 50  0000 L CNN
+F 0 "C$DDRn$135" V 7000 13450 50  0000 L CNN
+F 1 "0.1uF" H 7025 13050 50  0000 L CNN
 F 2 "Capacitors_SMD:C_0402" H 7000 13150 60  0001 C CNN
 F 3 "" H 7000 13150 60  0000 C CNN
@@
 U 1 1 57C6176F
 P 7400 13150
-F 0 "C$DDRn$137" H 7450 13250 50  0000 L CNN
-F 1 "0.1uF" H 7450 13050 50  0000 L CNN
+F 0 "C$DDRn$137" V 7400 13450 50  0000 L CNN
+F 1 "0.1uF" H 7425 13050 50  0000 L CNN
 F 2 "Capacitors_SMD:C_0402" H 7400 13150 60  0001 C CNN
 F 3 "" H 7400 13150 60  0000 C CNN
@@
 U 1 1 57C61770
 P 7800 13150
-F 0 "C$DDRn$139" H 7850 13250 50  0000 L CNN
-F 1 "0.1uF" H 7850 13050 50  0000 L CNN
+F 0 "C$DDRn$139" V 7800 13450 50  0000 L CNN
+F 1 "0.1uF" H 7825 13050 50  0000 L CNN
 F 2 "Capacitors_SMD:C_0402" H 7800 13150 60  0001 C CNN
 F 3 "" H 7800 13150 60  0000 C CNN
@@
 L C C$DDRn$141
 U 1 1 57C61771
-P 8100 13150
-F 0 "C$DDRn$141" H 8150 13250 50  0000 L CNN
-F 1 "0.1uF" H 8150 13050 50  0000 L CNN
-F 2 "Capacitors_SMD:C_0402" H 8100 13150 60  0001 C CNN
-F 3 "" H 8100 13150 60  0000 C CNN
-	1    8100 13150
+P 8175 13150
+F 0 "C$DDRn$141" V 8175 13450 50  0000 L CNN
+F 1 "0.1uF" H 8200 13050 50  0000 L CNN
+F 2 "Capacitors_SMD:C_0402" H 8175 13150 60  0001 C CNN
+F 3 "" H 8175 13150 60  0000 C CNN
+	1    8175 13150
 	-1   0    0    1
 $EndComp
@@
 L C C$DDRn$142
 U 1 1 57C61772
-P 8400 13150
-F 0 "C$DDRn$142" H 8450 13250 50  0000 L CNN
-F 1 "0.1uF" H 8450 13050 50  0000 L CNN
-F 2 "Capacitors_SMD:C_0402" H 8400 13150 60  0001 C CNN
-F 3 "" H 8400 13150 60  0000 C CNN
-	1    8400 13150
+P 8525 13150
+F 0 "C$DDRn$142" V 8525 13450 50  0000 L CNN
+F 1 "0.1uF" H 8550 13050 50  0000 L CNN
+F 2 "Capacitors_SMD:C_0402" H 8525 13150 60  0001 C CNN
+F 3 "" H 8525 13150 60  0000 C CNN
+	1    8525 13150
 	-1   0    0    1
 $EndComp
@@
 	7400 12850 7800 12850
 Wire Wire Line
-	7800 12850 8100 12850
-Wire Wire Line
-	8100 12850 8400 12850
-Wire Wire Line
-	8400 12850 8400 13000
+	7800 12850 8175 12850
+Wire Wire Line
+	8175 12850 8525 12850
+Wire Wire Line
+	8525 12850 8525 13000
 Wire Wire Line
 	2600 12850 2600 13000
@@
 Connection ~ 7800 12850
 Wire Wire Line
-	8100 13000 8100 12850
-Connection ~ 8100 12850
+	8175 13000 8175 12850
+Connection ~ 8175 12850
 Connection ~ 2250 12850
 Wire Bus Line
@@
 	7400 13400 7800 13400
 Wire Wire Line
-	7800 13400 8100 13400
-Wire Wire Line
-	8100 13400 8400 13400
-Wire Wire Line
-	3300 14550 3300 14650
-Wire Wire Line
-	3300 14650 3300 14800
+	7800 13400 8175 13400
+Wire Wire Line
+	8175 13400 8525 13400
+Wire Wire Line
+	8525 13400 8725 13400
+Wire Wire Line
+	2250 14650 2600 14650
+Wire Wire Line
+	2600 14650 2950 14650
+Wire Wire Line
+	2950 14650 3300 14650
+Wire Wire Line
+	3300 14650 3550 14650
 Wire Wire Line
 	2600 13300 2600 13400
@@
 Connection ~ 7800 13400
 Wire Wire Line
-	8100 13300 8100 13400
-Connection ~ 8100 13400
+	8175 13300 8175 13400
+Connection ~ 8175 13400
 Text Label 9500 5250 0    60   ~ 0
 GND
@@
 L GND #PWR101
 U 1 1 57DC0DED
-P 3300 14800
-F 0 "#PWR101" H 3300 14800 30  0001 C CNN
-F 1 "GND" H 3300 14730 30  0001 C CNN
-F 2 "" H 3300 14800 60  0000 C CNN
-F 3 "" H 3300 14800 60  0000 C CNN
-	1    3300 14800
-	1    0    0    -1
-$EndComp
-Text Label 3300 14800 0    60   ~ 0
+P 3550 14650
+F 0 "#PWR101" H 3550 14650 30  0001 C CNN
+F 1 "GND" H 3550 14580 30  0001 C CNN
+F 2 "" H 3550 14650 60  0000 C CNN
+F 3 "" H 3550 14650 60  0000 C CNN
+	1    3550 14650
+	0    -1   -1   0
+$EndComp
+Text Label 3550 14650 1    60   ~ 0
 GND
 $Comp
@@
 U 1 1 57DC201F
 P 2250 14400
-F 0 "C$DDRn$101" H 2300 14500 50  0000 L CNN
-F 1 "0.1uF" H 2300 14300 50  0000 L CNN
+F 0 "C$DDRn$101" V 2250 14700 50  0000 L CNN
+F 1 "0.1uF" H 2275 14325 50  0000 L CNN
 F 2 "Capacitors_SMD:C_0402" H 2250 14400 60  0001 C CNN
 F 3 "" H 2250 14400 60  0000 C CNN
@@
 U 1 1 57DC2489
 P 2600 14400
-F 0 "C$DDRn$103" H 2650 14500 50  0000 L CNN
-F 1 "0.1uF" H 2650 14300 50  0000 L CNN
+F 0 "C$DDRn$103" V 2600 14700 50  0000 L CNN
+F 1 "0.1uF" H 2625 14325 50  0000 L CNN
 F 2 "Capacitors_SMD:C_0402" H 2600 14400 60  0001 C CNN
 F 3 "" H 2600 14400 60  0000 C CNN
@@
 U 1 1 57DC2506
 P 3300 14400
-F 0 "C$DDRn$106" H 3350 14500 50  0000 L CNN
-F 1 "0.1uF" H 3350 14300 50  0000 L CNN
+F 0 "C$DDRn$106" V 3300 14700 50  0000 L CNN
+F 1 "0.1uF" H 3325 14325 50  0000 L CNN
 F 2 "Capacitors_SMD:C_0402" H 3300 14400 60  0001 C CNN
 F 3 "" H 3300 14400 60  0000 C CNN
@@
 U 1 1 57DC26FE
 P 2950 14400
-F 0 "C$DDRn$104" H 3000 14500 50  0000 L CNN
-F 1 "0.1uF" H 3000 14300 50  0000 L CNN
+F 0 "C$DDRn$104" V 2950 14700 50  0000 L CNN
+F 1 "0.1uF" H 2975 14325 50  0000 L CNN
 F 2 "Capacitors_SMD:C_0402" H 2950 14400 60  0001 C CNN
 F 3 "" H 2950 14400 60  0000 C CNN
@@
 Wire Wire Line
 	2250 14550 2250 14650
-Wire Wire Line
-	2250 14650 2600 14650
-Wire Wire Line
-	2600 14650 2950 14650
-Wire Wire Line
-	2950 14650 3300 14650
 Connection ~ 3300 14650
 Wire Wire Line
@@
 Wire Wire Line
 	10150 5150 10150 5100
-Text Notes 10250 4400 0    60   ~ 0
+Text Notes 10275 4450 0    60   ~ 0
 CA Bypass
-Text Notes 10300 4950 0    60   ~ 0
+Text Notes 10275 4975 0    60   ~ 0
 DQ Bypass\n
 Wire Wire Line
 	10150 4000 10150 4250
 Wire Wire Line
-	8400 13300 8400 13550
+	8525 13400 8525 13300
 $Comp
 L R R$DDRn$102
@@
 L GND #PWR?
 U 1 1 57DBC649
-P 8400 13550
-F 0 "#PWR?" H 8400 13550 30  0001 C CNN
-F 1 "GND" H 8400 13480 30  0001 C CNN
-F 2 "" H 8400 13550 60  0000 C CNN
-F 3 "" H 8400 13550 60  0000 C CNN
-	1    8400 13550
-	1    0    0    -1
-$EndComp
-Text Label 8400 13550 0    60   ~ 0
+P 8725 13400
+F 0 "#PWR?" H 8725 13400 30  0001 C CNN
+F 1 "GND" H 8725 13330 30  0001 C CNN
+F 2 "" H 8725 13400 60  0000 C CNN
+F 3 "" H 8725 13400 60  0000 C CNN
+	1    8725 13400
+	0    -1   -1   0
+$EndComp
+Text Label 8675 13400 1    60   ~ 0
 GND
 Text Label 11650 4750 2    60   ~ 0
@@
 Text Label 1550 14150 0    60   ~ 0
 $DDRn$10V75
+Connection ~ 8525 13400
+Wire Wire Line
+	3300 14650 3300 14550
 $EndSCHEMATC
